File: bee-light-measurement-matrix.sch (KiCad schematic (older format))
At the start: 35 parts, among them P1 CONN_01X10, U1 MCP3208, U2 MCP3208

Commit message: Update of the schematics
Parts:
- removed P1: CONN_01X10, symbol CONN_01X10
- removed R1, R17, R18, R19, R2, R20, R21, R22, R23, R24, R5, R6, R7, R8: R, symbol R
- added C1, C2, C4: 100n, Capacitors_THT:C_Disc_D7.0mm_W2.5mm_P5.00mm, symbol C
- added C3: 10µ, Capacitors_THT:CP_Radial_Tantal_D4.5mm_P5.00mm, symbol CP
- added J1: CONN_02X13, Pin_Headers:Pin_Header_Straight_2x13_Pitch2.54mm, symbol CONN_02X13
- added J3: CONN_01X03, Pin_Headers:Pin_Header_Straight_1x03_Pitch2.54mm, symbol CONN_01X03
- added J4: CONN_02X10, Pin_Headers:Pin_Header_Straight_2x10_Pitch2.54mm, symbol CONN_02X10
- added RN1, RN2: R_Network08, Resistors_THT:R_Array_SIP9, symbol R_Network08
- added U3: MCP1541, TO_SOT_Packages_THT:TO-92_Molded_Narrow, symbol MCP1541-RESCUE-bee-light-measurement-matrix
- R1.1: renamed from R16; footprint (none) -> Discret:R1
- R1.2: renamed from R15; footprint (none) -> Discret:R1
- R1.3: renamed from R14; footprint (none) -> Discret:R1
- R1.4: renamed from R13; footprint (none) -> Discret:R1
- R1.5: renamed from R12; footprint (none) -> Discret:R1
- R1.6: renamed from R11; footprint (none) -> Discret:R1
- R1.7: renamed from R10; footprint (none) -> Discret:R1
- R1.8: renamed from R9; footprint (none) -> Discret:R1
- R2.1: renamed from R32; footprint (none) -> Discret:R1
- R2.2: renamed from R31; footprint (none) -> Discret:R1
- R2.3: renamed from R30; footprint (none) -> Discret:R1
- R2.4: renamed from R29; footprint (none) -> Discret:R1
- R2.5: renamed from R28; footprint (none) -> Discret:R1
- R2.6: renamed from R27; footprint (none) -> Discret:R1
- R2.7: renamed from R26; footprint (none) -> Discret:R1
- R2.8: renamed from R25; footprint (none) -> Discret:R1
- R3, R4: value R -> 100k; footprint (none) -> Resistors_THT:R_Axial_DIN0414_L11.9mm_D4.5mm_P5.08mm_Vertical
- U1, U2: footprint (none) -> Housings_DIP:DIP-16_W7.62mm
Connections:
- net GND: now also C1.2, C2.2, C3.2, C4.1, J1.14 (P14), J1.20 (P20), J1.25 (P25), J1.6 (P6), J1.9 (P9), J3.1 (P1), J4.1 (P1), J4.2 (P2), U3.1 (GND)
- net at R1.1.1, U1.1 (CH0): now also J4.3 (P3), RN1.9 (R8)
- net CE0: now reaches U1.10 (~CS)
- net CE0: now also R3.2, J1.24 (P24)
- net MOSI: now reaches U1.11 (Din), U2.11 (Din)
- net MOSI: now also J1.19 (P19)
- net MISO: now reaches U1.12 (Dout), U2.12 (Dout)
- net MISO: now also J1.21 (P21)
- net CLK: now reaches U1.13 (CLK), U2.13 (CLK)
- net CLK: now also J1.23 (P23)
- net at R1.2.1, U1.2 (CH1): now also J4.5 (P5), RN1.8 (R7)
- net at R1.3.1, U1.3 (CH2): now also J4.7 (P7), RN1.7 (R6)
- net at R1.4.1, U1.4 (CH3): now also J4.9 (P9), RN1.6 (R5)
- net at R1.5.1, U1.5 (CH4): now also J4.11 (P11), RN1.5 (R4); no longer R4.2
- net at R1.6.1, U1.6 (CH5): now also J4.13 (P13), RN1.4 (R3); no longer R3.2
- net at R1.7.1, U1.7 (CH6): now also J4.15 (P15), RN1.3 (R2)
- net at R1.8.1, U1.8 (CH7): now also J4.17 (P17), RN1.2 (R1)
- net at R2.1.1, U2.1 (CH0): now also J4.4 (P4), RN2.9 (R8)
- net CE1: now reaches U2.10 (~CS)
- net CE1: now also R4.2, J1.26 (P26)
- net at R2.2.1, U2.2 (CH1): now also J4.6 (P6), RN2.8 (R7)
- net at R2.3.1, U2.3 (CH2): now also J4.8 (P8), RN2.7 (R6)
- net at R2.4.1, U2.4 (CH3): now also J4.10 (P10), RN2.6 (R5)
- net at R2.5.1, U2.5 (CH4): now also J4.12 (P12), RN2.5 (R4)
- net at R2.6.1, U2.6 (CH5): now also J4.14 (P14), RN2.4 (R3)
- net at R2.7.1, U2.7 (CH6): now also J4.16 (P16), RN2.3 (R2)
- net at R2.8.1, U2.8 (CH7): now also J4.18 (P18), RN2.2 (R1)
- net +3V3 renamed +5V
- net +5V: now also C1.1, C2.1, C3.1, C4.2, J1.2 (P2), RN1.1 (common), RN2.1 (common), U3.3 (Vin); no longer U1.15 (Vref), U2.15 (Vref)
- new net GPIO25: J1.22 (P22)
- new net RXD: J1.10 (P10), J3.3 (P3)
- new net TXD: J1.8 (P8), J3.2 (P2)
- new net Vref: U1.15 (Vref), U2.15 (Vref), U3.2 (Vout)
- no-connect marks 3 -> 14
Other:
- note added: "LDR Connector"
- note added: "Referenz\nVoltage"
- note added: "TTL COM\nConnector"
- note added: "schematic based on\nhttp://www.raspberrypi-spy.co.uk/2013/10/analogue-sensors-on-the-raspberry-pi-using-an-mcp3008/"
- note removed: "CS1"
- note removed: "CS2"
- note removed: "Clock"
- note removed: "MISO"
- note removed: "MOSI"
- note removed: "based on\nhttp://www.raspberrypi-spy.co.uk/2013/10/analogue-sensors-on-the-raspberry-pi-using-an-mcp3008/"
- moved on the sheet: R1.1, R1.2, R1.3, R1.4, R1.5, R1.6, R1.7, R1.8, R2.1, R2.2, R2.3, R2.4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
